File: analog_filters.sch (KiCad schematic (older format))
At the start: 0 parts

Commit message: Files from laptop
Parts:
- added C? (x4): 1uF, symbol C_Small
- added J? (x4): PAD, part_footprints:SOLDER_PAD, symbol PAD
- added R? (x4): 49.9K, symbol R_Small
Connections:
- net AIN_1: now also C?.1, R?.1
- net AIN_2: now also C?.1, R?.1
- net AIN_3: now also C?.1, R?.1
- new net: J?.1, R?.2 (x4)
- new net AIN_0: C?.1, R?.1
- new net GND: C?.2, C?.2, C?.2, C?.2
Changed lines of the file:
@@
 Comment4 ""
 $EndDescr
-Text HLabel 7750 3250 2    60   Output ~ 0
+Text HLabel 3950 2050 2    60   Output ~ 0
+AIN_0
+Text HLabel 3950 3000 2    60   Output ~ 0
 AIN_1
-Text HLabel 7750 3450 2    60   Output ~ 0
+Text HLabel 3950 3950 2    60   Output ~ 0
 AIN_2
-Text HLabel 7750 3650 2    60   Output ~ 0
+$Comp
+L R_Small R?
+U 1 1 5A3C8A6D
+P 3200 2050
+F 0 "R?" V 3100 2000 50  0000 L CNN
+F 1 "49.9K" V 3300 1950 50  0000 L CNN
+F 2 "" H 3200 2050 50  0001 C CNN
+F 3 "" H 3200 2050 50  0001 C CNN
+	1    3200 2050
+	0    1    1    0
+$EndComp
+$Comp
+L PAD J?
+U 1 1 5A3C8B0A
+P 2650 2050
+F 0 "J?" H 2750 2050 60  0000 C CNN
+F 1 "PAD" H 2650 1950 60  0001 C CNN
+F 2 "part_footprints:SOLDER_PAD" H 2650 1950 60  0001 C CNN
+F 3 "" H 2750 2050 60  0001 C CNN
+	1    2650 2050
+	-1   0    0    1
+$EndComp
+Wire Wire Line
+	2750 2050 3100 2050
+$Comp
+L C_Small C?
+U 1 1 5A3C8B90
+P 3600 2250
+F 0 "C?" H 3610 2320 50  0000 L CNN
+F 1 "1uF" H 3610 2170 50  0000 L CNN
+F 2 "" H 3600 2250 50  0001 C CNN
+F 3 "" H 3600 2250 50  0001 C CNN
+	1    3600 2250
+	1    0    0    -1
+$EndComp
+$Comp
+L GND #PWR?
+U 1 1 5A3C8BB7
+P 3600 2500
+F 0 "#PWR?" H 3600 2250 50  0001 C CNN
+F 1 "GND" H 3600 2350 50  0000 C CNN
+F 2 "" H 3600 2500 50  0001 C CNN
+F 3 "" H 3600 2500 50  0001 C CNN
+	1    3600 2500
+	1    0    0    -1
+$EndComp
+Wire Wire Line
+	3600 2500 3600 2350
+Wire Wire Line
+	3300 2050 3950 2050
+Wire Wire Line
+	3600 2050 3600 2150
+Connection ~ 3600 2050
+$Comp
+L R_Small R?
+U 1 1 5A3C8D5A
+P 3200 3000
+F 0 "R?" V 3100 2950 50  0000 L CNN
+F 1 "49.9K" V 3300 2900 50  0000 L CNN
+F 2 "" H 3200 3000 50  0001 C CNN
+F 3 "" H 3200 3000 50  0001 C CNN
+	1    3200 3000
+	0    1    1    0
+$EndComp
+$Comp
+L PAD J?
+U 1 1 5A3C8D60
+P 2650 3000
+F 0 "J?" H 2750 3000 60  0000 C CNN
+F 1 "PAD" H 2650 2900 60  0001 C CNN
+F 2 "part_footprints:SOLDER_PAD" H 2650 2900 60  0001 C CNN
+F 3 "" H 2750 3000 60  0001 C CNN
+	1    2650 3000
+	-1   0    0    1
+$EndComp
+Wire Wire Line
+	2750 3000 3100 3000
+$Comp
+L C_Small C?
+U 1 1 5A3C8D67
+P 3600 3200
+F 0 "C?" H 3610 3270 50  0000 L CNN
+F 1 "1uF" H 3610 3120 50  0000 L CNN
+F 2 "" H 3600 3200 50  0001 C CNN
+F 3 "" H 3600 3200 50  0001 C CNN
+	1    3600 3200
+	1    0    0    -1
+$EndComp
+$Comp
+L GND #PWR?
+U 1 1 5A3C8D6D
+P 3600 3450
+F 0 "#PWR?" H 3600 3200 50  0001 C CNN
+F 1 "GND" H 3600 3300 50  0000 C CNN
+F 2 "" H 3600 3450 50  0001 C CNN
+F 3 "" H 3600 3450 50  0001 C CNN
+	1    3600 3450
+	1    0    0    -1
+$EndComp
+Wire Wire Line
+	3600 3450 3600 3300
+Wire Wire Line
+	3300 3000 3950 3000
+Wire Wire Line
+	3600 3000 3600 3100
+Connection ~ 3600 3000
+$Comp
+L R_Small R?
+U 1 1 5A3C8EF4
+P 3200 3950
+F 0 "R?" V 3100 3900 50  0000 L CNN
+F 1 "49.9K" V 3300 3850 50  0000 L CNN
+F 2 "" H 3200 3950 50  0001 C CNN
+F 3 "" H 3200 3950 50  0001 C CNN
+	1    3200 3950
+	0    1    1    0
+$EndComp
+$Comp
+L PAD J?
+U 1 1 5A3C8EFA
+P 2650 3950
+F 0 "J?" H 2750 3950 60  0000 C CNN
+F 1 "PAD" H 2650 3850 60  0001 C CNN
+F 2 "part_footprints:SOLDER_PAD" H 2650 3850 60  0001 C CNN
+F 3 "" H 2750 3950 60  0001 C CNN
+	1    2650 3950
+	-1   0    0    1
+$EndComp
+Wire Wire Line
+	2750 3950 3100 3950
+$Comp
+L C_Small C?
+U 1 1 5A3C8F01
+P 3600 4150
+F 0 "C?" H 3610 4220 50  0000 L CNN
+F 1 "1uF" H 3610 4070 50  0000 L CNN
+F 2 "" H 3600 4150 50  0001 C CNN
+F 3 "" H 3600 4150 50  0001 C CNN
+	1    3600 4150
+	1    0    0    -1
+$EndComp
+$Comp
+L GND #PWR?
+U 1 1 5A3C8F07
+P 3600 4400
+F 0 "#PWR?" H 3600 4150 50  0001 C CNN
+F 1 "GND" H 3600 4250 50  0000 C CNN
+F 2 "" H 3600 4400 50  0001 C CNN
+F 3 "" H 3600 4400 50  0001 C CNN
+	1    3600 4400
+	1    0    0    -1
+$EndComp
+Wire Wire Line
+	3600 4400 3600 4250
+Wire Wire Line
+	3300 3950 3950 3950
+Wire Wire Line
+	3600 3950 3600 4050
+Connection ~ 3600 3950
+$Comp
+L R_Small R?
+U 1 1 5A3C97A0
+P 3200 4950
+F 0 "R?" V 3100 4900 50  0000 L CNN
+F 1 "49.9K" V 3300 4850 50  0000 L CNN
+F 2 "" H 3200 4950 50  0001 C CNN
+F 3 "" H 3200 4950 50  0001 C CNN
+	1    3200 4950
+	0    1    1    0
+$EndComp
+$Comp
+L PAD J?
+U 1 1 5A3C97A6
+P 2650 4950
+F 0 "J?" H 2750 4950 60  0000 C CNN
+F 1 "PAD" H 2650 4850 60  0001 C CNN
+F 2 "part_footprints:SOLDER_PAD" H 2650 4850 60  0001 C CNN
+F 3 "" H 2750 4950 60  0001 C CNN
+	1    2650 4950
+	-1   0    0    1
+$EndComp
+Wire Wire Line
+	2750 4950 3100 4950
+$Comp
+L C_Small C?
+U 1 1 5A3C97AD
+P 3600 5150
+F 0 "C?" H 3610 5220 50  0000 L CNN
+F 1 "1uF" H 3610 5070 50  0000 L CNN
+F 2 "" H 3600 5150 50  0001 C CNN
+F 3 "" H 3600 5150 50  0001 C CNN
+	1    3600 5150
+	1    0    0    -1
+$EndComp
+$Comp
+L GND #PWR?
+U 1 1 5A3C97B3
+P 3600 5400
+F 0 "#PWR?" H 3600 5150 50  0001 C CNN
+F 1 "GND" H 3600 5250 50  0000 C CNN
+F 2 "" H 3600 5400 50  0001 C CNN
+F 3 "" H 3600 5400 50  0001 C CNN
+	1    3600 5400
+	1    0    0    -1
+$EndComp
+Wire Wire Line
+	3600 5400 3600 5250
+Wire Wire Line
+	3300 4950 3950 4950
+Wire Wire Line
+	3600 4950 3600 5050
+Connection ~ 3600 4950
+Text HLabel 3950 4950 2    60   Output ~ 0
 AIN_3
 $EndSCHEMATC
