File: esp8266.sch (KiCad schematic (older format))
At the start: 0 parts

Commit message: Files from laptop
Parts:
- added C? (x2): 0.1uF, symbol C_Small
- added C?: 10uF, symbol C_Small
- added R? (x4): 10K, symbol R_Small
- added U?: ESP-13-WROOM-02, part_footprints:ESP-13-WROOM-02, symbol ESP-13-WROOM-02
Connections:
- net BOOTLOADER: now also R?.2, U?.8 (GPIO0)
- net RX: now also U?.11 (RXD)
- net TX: now also U?.12 (TXD)
- net WAKE: now also R?.2, U?.15 (~RST~)
- new net: C?.1, R?.2, U?.2 (EN)
- new net: R?.1, U?.6 (GPIO15)
- new net GND: C?.2, C?.2, C?.2, R?.2, U?.13 (GND), U?.18 (GND), U?.9 (GND), U?.PAD (GND)
- new net VDD: C?.1, C?.1, R?.1, R?.1, R?.1, U?.1 (VCC)
Other:
- note added: "DEPOP"
- note added: "Ensure RST and BOOTLOADER\nare high during boot"
- note added: "use EN instead of WAKE?"
