File: i2c_peripherals.sch (KiCad schematic (older format))
At the start: 0 parts

Commit message: Files from laptop
Parts:
- added C? (x3): 0.1uF, symbol C_Small
- added U?: SI7021-A20, part_footprints:DFN-6-1EP_3x3mm_Pitch1.00mm, symbol SI7021-A20
- added U?: 24FC64FT, symbol 24FC64FT
- added U?: VEML7700, part_footprints:VEML7700, symbol VEML7700
Connections:
- net SCL: now also U?.1 (SCL), U?.1 (SCL), U?.6 (SCL)
- net SDA: now also U?.1 (SDA), U?.3 (SDA), U?.4 (SDA)
- new net GND: C?.2, C?.2, C?.2, U?.2 (GND), U?.2 (GND), U?.3 (GND), U?.5 (WP)
- new net VDD: C?.1, C?.1, C?.1, U?.2 (VDD), U?.4 (VCC), U?.5 (VDD)
Other:
- note added: "EEPROM"
- note added: "Lux meter"
- note added: "Temp/humidity"
Changed lines of the file:
@@
 Comment4 ""
 $EndDescr
-Text HLabel 1750 2600 0    60   BiDi ~ 0
+Text HLabel 3450 1900 0    60   BiDi ~ 0
 SDA
-Text HLabel 1750 2800 0    60   BiDi ~ 0
+Text HLabel 3450 1800 0    60   BiDi ~ 0
 SCL
+$Comp
+L SI7021-A20 U?
+U 1 1 5A3DD81C
+P 4000 1900
+F 0 "U?" H 4100 2225 60  0000 C CNN
+F 1 "SI7021-A20" H 4000 1550 60  0000 C CNN
+F 2 "part_footprints:DFN-6-1EP_3x3mm_Pitch1.00mm" H 4000 1450 60  0001 C CNN
+F 3 "" H 4000 1900 60  0001 C CNN
+	1    4000 1900
+	1    0    0    -1
+$EndComp
+$Comp
+L 24FC64FT U?
+U 1 1 5A3DD845
+P 3950 3600
+F 0 "U?" H 4100 3950 60  0000 C CNN
+F 1 "24FC64FT" H 3925 3325 60  0000 C CNN
+F 2 "" H 3950 3600 60  0001 C CNN
+F 3 "" H 3950 3600 60  0001 C CNN
+	1    3950 3600
+	1    0    0    -1
+$EndComp
+$Comp
+L VEML7700 U?
+U 1 1 5A3DD8CE
+P 7800 2600
+F 0 "U?" H 8150 2900 60  0000 C CNN
+F 1 "VEML7700" H 7650 2300 60  0000 C CNN
+F 2 "part_footprints:VEML7700" H 7800 2200 60  0001 C CNN
+F 3 "" H 7800 2600 60  0001 C CNN
+	1    7800 2600
+	1    0    0    -1
+$EndComp
+Text HLabel 3300 3500 0    60   BiDi ~ 0
+SDA
+Text HLabel 3300 3400 0    60   BiDi ~ 0
+SCL
+Text HLabel 7000 2700 0    60   BiDi ~ 0
+SDA
+Text HLabel 7000 2500 0    60   BiDi ~ 0
+SCL
+Wire Wire Line
+	3450 1800 3600 1800
+Wire Wire Line
+	3600 1900 3450 1900
+Wire Wire Line
+	3300 3400 3500 3400
+Wire Wire Line
+	3500 3500 3300 3500
+Wire Wire Line
+	7000 2500 7200 2500
+Wire Wire Line
+	7200 2700 7000 2700
+$Comp
+L C_Small C?
+U 1 1 5A3DDB04
+P 4550 1900
+F 0 "C?" H 4560 1970 50  0000 L CNN
+F 1 "0.1uF" H 4560 1820 50  0000 L CNN
+F 2 "" H 4550 1900 50  0001 C CNN
+F 3 "" H 4550 1900 50  0001 C CNN
+	1    4550 1900
+	1    0    0    -1
+$EndComp
+$Comp
+L GND #PWR?
+U 1 1 5A3DDB2B
+P 4550 2200
+F 0 "#PWR?" H 4550 1950 50  0001 C CNN
+F 1 "GND" H 4550 2050 50  0000 C CNN
+F 2 "" H 4550 2200 50  0001 C CNN
+F 3 "" H 4550 2200 50  0001 C CNN
+	1    4550 2200
+	1    0    0    -1
+$EndComp
+$Comp
+L VDD #PWR?
+U 1 1 5A3DDB47
+P 4550 1600
+F 0 "#PWR?" H 4550 1450 50  0001 C CNN
+F 1 "VDD" H 4550 1750 50  0000 C CNN
+F 2 "" H 4550 1600 50  0001 C CNN
+F 3 "" H 4550 1600 50  0001 C CNN
+	1    4550 1600
+	1    0    0    -1
+$EndComp
+Wire Wire Line
+	4400 1700 4550 1700
+Wire Wire Line
+	4550 1600 4550 1800
+Connection ~ 4550 1700
+Wire Wire Line
+	4550 2200 4550 2000
+Wire Wire Line
+	4400 2100 4550 2100
+Connection ~ 4550 2100
+$Comp
+L C_Small C?
+U 1 1 5A3DDC28
+P 4700 3550
+F 0 "C?" H 4710 3620 50  0000 L CNN
+F 1 "0.1uF" H 4710 3470 50  0000 L CNN
+F 2 "" H 4700 3550 50  0001 C CNN
+F 3 "" H 4700 3550 50  0001 C CNN
+	1    4700 3550
+	1    0    0    -1
+$EndComp
+$Comp
+L GND #PWR?
+U 1 1 5A3DDC2E
+P 4700 3850
+F 0 "#PWR?" H 4700 3600 50  0001 C CNN
+F 1 "GND" H 4700 3700 50  0000 C CNN
+F 2 "" H 4700 3850 50  0001 C CNN
+F 3 "" H 4700 3850 50  0001 C CNN
+	1    4700 3850
+	1    0    0    -1
+$EndComp
+$Comp
+L VDD #PWR?
+U 1 1 5A3DDC34
+P 4700 3250
+F 0 "#PWR?" H 4700 3100 50  0001 C CNN
+F 1 "VDD" H 4700 3400 50  0000 C CNN
+F 2 "" H 4700 3250 50  0001 C CNN
+F 3 "" H 4700 3250 50  0001 C CNN
+	1    4700 3250
+	1    0    0    -1
+$EndComp
+Wire Wire Line
+	4700 3250 4700 3450
+Wire Wire Line
+	4700 3650 4700 3850
+Wire Wire Line
+	4400 3400 4700 3400
+Connection ~ 4700 3400
+Wire Wire Line
+	4400 3700 4700 3700
+Connection ~ 4700 3700
+Wire Wire Line
+	4400 3600 4500 3600
+Wire Wire Line
+	4500 3600 4500 3700
+Connection ~ 4500 3700
+$Comp
+L C_Small C?
+U 1 1 5A3DDEC4
+P 8800 2600
+F 0 "C?" H 8810 2670 50  0000 L CNN
+F 1 "0.1uF" H 8810 2520 50  0000 L CNN
+F 2 "" H 8800 2600 50  0001 C CNN
+F 3 "" H 8800 2600 50  0001 C CNN
+	1    8800 2600
+	1    0    0    -1
+$EndComp
+$Comp
+L GND #PWR?
+U 1 1 5A3DDECA
+P 8800 2900
+F 0 "#PWR?" H 8800 2650 50  0001 C CNN
+F 1 "GND" H 8800 2750 50  0000 C CNN
+F 2 "" H 8800 2900 50  0001 C CNN
+F 3 "" H 8800 2900 50  0001 C CNN
+	1    8800 2900
+	1    0    0    -1
+$EndComp
+$Comp
+L VDD #PWR?
+U 1 1 5A3DDED0
+P 8800 2300
+F 0 "#PWR?" H 8800 2150 50  0001 C CNN
+F 1 "VDD" H 8800 2450 50  0000 C CNN
+F 2 "" H 8800 2300 50  0001 C CNN
+F 3 "" H 8800 2300 50  0001 C CNN
+	1    8800 2300
+	1    0    0    -1
+$EndComp
+Wire Wire Line
+	8800 2300 8800 2500
+Wire Wire Line
+	8800 2700 8800 2900
+Wire Wire Line
+	8500 2450 8800 2450
+Connection ~ 8800 2450
+Wire Wire Line
+	8500 2750 8800 2750
+Connection ~ 8800 2750
+Wire Wire Line
+	8400 2500 8500 2500
+Wire Wire Line
+	8500 2500 8500 2450
+Wire Wire Line
+	8500 2750 8500 2700
+Wire Wire Line
+	8500 2700 8400 2700
+Text Notes 7500 2100 0    60   ~ 0
+Lux meter
+Text Notes 3700 1250 0    60   ~ 0
+Temp/humidity
+Text Notes 3800 3050 0    60   ~ 0
+EEPROM
 $EndSCHEMATC
