File: power.sch (KiCad schematic (older format))
At the start: 11 parts

Commit message: Files from laptop
Connections:
- net VSYS: no longer names the net of C?.1, D?.1 (K), Q?.2 (S), U?.1 (VIN), U?.2 (INPUT)
Other:
- note added: "3.0V Regulated"
Changed lines of the file:
@@
 Wire Wire Line
 	4550 2600 4450 2600
-Wire Wire Line
-	4450 2050 4450 3550
 Connection ~ 4450 2200
 Wire Wire Line
@@
 VUSB
 Wire Wire Line
-	4450 2050 4600 2050
-Text HLabel 4600 2050 2    60   Output ~ 0
-VSYS
+	4450 2200 4450 3550
+Text Notes 8000 2100 0    60   ~ 0
+3.0V Regulated
 $EndSCHEMATC
