File: stm32l051k8t.sch (KiCad schematic (older format))
At the start: 0 parts

Commit message: Files from laptop
Parts:
- added C? (x4): 0.1uF, symbol C_Small
- added C?: 10uF, symbol C_Small
- added C?: 1.0uF, symbol C_Small
- added J?: Conn_01x04, symbol Conn_01x04
- added R? (x2): 2.2K, symbol R_Small
- added R?: 10K, symbol R_Small
- added U?: STM32L051K8T6, part_footprints:LQFP-32_7x7mm_Pitch0.8mm, symbol STM32L051K8T6
Connections:
- net AIN_0: now also U?.6 (PA0)
- net AIN_1: now also U?.7 (PA1)
- net AIN_2: now also U?.8 (PA2)
- net AIN_3: now also U?.9 (PA3)
- net BOOTLOADER: now also R?.1, U?.31 (BOOT0)
- net ESP_WAKE: now also U?.18 (PA8)
- net OPTO_0: now also U?.28 (PB5)
- net OPTO_1: now also U?.27 (PB4)
- net OPTO_2: now also U?.26 (PB3)
- net OPTO_3: now also U?.22 (PA12)
- net SCL: now also R?.2, U?.29 (PB6)
- net SDA: now also R?.2, U?.30 (PB7)
- net SW_0: now also U?.14 (PB0)
- net SW_1: now also U?.15 (PB1)
- net USART1_RX: now also U?.20 (PA10)
- net USART1_TX: now also U?.19 (PA9)
- net USART2_RX: now also U?.25 (PA15)
- net USART2_TX: now also U?.24 (PA14)
- new net GND: C?.2, C?.2, C?.2, C?.2, C?.2, C?.2, R?.2, U?.16 (VSS), U?.32 (VSS)
- new net PA4: U?.10 (PA4)
- new net PA5: U?.11 (PA5)
- new net SYS_SWDIO: U?.23 (PA13)
- new net VDD: C?.1, C?.1, C?.1, C?.1, C?.1, R?.1, R?.1, U?.1 (VDD), U?.17 (VDD), U?.5 (VDDA)
- new net ~RST: C?.1, U?.4 (NRST)
Other:
- note added: "0.1uF for each and 10uF for one VDD\n0.1uF and 1uF for VDDA"
- note added: "Ensure BOOTLOADER pin is 0 during boot"
- note added: "ST-LINK"
- note added: "~RST~ has internal pull-up"
