File: usb_serial.sch (KiCad schematic (older format))
At the start: 0 parts

Commit message: Files from laptop
Parts:
- added C? (x2): 0.1uF, symbol C_Small
- added C? (x2): 4.7uF, symbol C_Small
- added R?: 1K, symbol R_Small
- added U?: CP2102N-A01-GQFN24, Housings_DFN_QFN:QFN-24-1EP_4x4mm_Pitch0.5mm, symbol CP2102N-A01-GQFN24
- added U?: SP0503BAHTG, TO_SOT_Packages_SMD:SOT-143, symbol SP0503BAHTG
Connections:
- net D+: now also U?.2, U?.3 (D+)
- net D-: now also U?.3, U?.4 (D-)
- net RX: now also U?.20 (RXD)
- net STM_BL: now also U?.14 (GPIO.0)
- net TX: now also U?.21 (TXD)
- net VUSB: now also C?.1, C?.1, U?.4, U?.7 (REGIN), U?.8 (VBUS)
- new net: R?.2, U?.9 (~RSTb)
- new net 3.3V_USB: C?.1, C?.1, R?.1, U?.5 (VIO), U?.6 (VDD)
- new net ESP_BL: U?.12 (GPIO.2)
- new net GND: C?.2, C?.2, C?.2, C?.2, U?.1, U?.2 (GND), U?.25 (GND)
- new net STM_~RST~: U?.13 (GPIO.1)
Changed lines of the file:
@@
 Comment4 ""
 $EndDescr
-Text HLabel 1800 2050 0    60   BiDi ~ 0
+Text HLabel 4350 3500 0    60   BiDi ~ 0
 D+
-Text HLabel 1800 2200 0    60   BiDi ~ 0
+Text HLabel 4350 3600 0    60   BiDi ~ 0
 D-
-Text HLabel 2850 2050 2    60   Output ~ 0
+Text HLabel 6300 2900 2    60   Output ~ 0
 TX
-Text HLabel 2850 2200 2    60   Input ~ 0
+Text HLabel 6300 2800 2    60   Input ~ 0
 RX
-Text HLabel 2850 2350 2    60   Output ~ 0
+Text HLabel 6300 3700 2    60   Output ~ 0
 STM_BL
-Text HLabel 1800 2400 0    60   Input ~ 0
+Text HLabel 3100 3100 0    60   Input ~ 0
 VUSB
+Text HLabel 6300 3500 2    60   Output ~ 0
+ESP_BL
+Text HLabel 6300 3600 2    60   Output ~ 0
+STM_~RST~
+$Comp
+L CP2102N-A01-GQFN24 U?
+U 1 1 5A428FD0
+P 5500 3100
+F 0 "U?" H 5900 3900 50  0000 R CNN
+F 1 "CP2102N-A01-GQFN24" H 6650 2250 50  0000 R CNN
+F 2 "Housings_DFN_QFN:QFN-24-1EP_4x4mm_Pitch0.5mm" H 5950 2300 50  0001 L CNN
+F 3 "" H 5550 2050 50  0001 C CNN
+	1    5500 3100
+	1    0    0    -1
+$EndComp
+$Comp
+L R_Small R?
+U 1 1 5A429094
+P 4550 2350
+F 0 "R?" H 4580 2370 50  0000 L CNN
+F 1 "1K" H 4580 2310 50  0000 L CNN
+F 2 "" H 4550 2350 50  0001 C CNN
+F 3 "" H 4550 2350 50  0001 C CNN
+	1    4550 2350
+	1    0    0    -1
+$EndComp
+$Comp
+L C_Small C?
+U 1 1 5A4290E6
+P 5650 1800
+F 0 "C?" H 5660 1870 50  0000 L CNN
+F 1 "0.1uF" H 5660 1720 50  0000 L CNN
+F 2 "" H 5650 1800 50  0001 C CNN
+F 3 "" H 5650 1800 50  0001 C CNN
+	1    5650 1800
+	1    0    0    -1
+$EndComp
+$Comp
+L C_Small C?
+U 1 1 5A42915C
+P 6100 1800
+F 0 "C?" H 6110 1870 50  0000 L CNN
+F 1 "4.7uF" H 6110 1720 50  0000 L CNN
+F 2 "" H 6100 1800 50  0001 C CNN
+F 3 "" H 6100 1800 50  0001 C CNN
+	1    6100 1800
+	1    0    0    -1
+$EndComp
+$Comp
+L GND #PWR?
+U 1 1 5A42927F
+P 6100 2050
+F 0 "#PWR?" H 6100 1800 50  0001 C CNN
+F 1 "GND" H 6100 1900 50  0000 C CNN
+F 2 "" H 6100 2050 50  0001 C CNN
+F 3 "" H 6100 2050 50  0001 C CNN
+	1    6100 2050
+	1    0    0    -1
+$EndComp
+Text Label 5750 1650 0    60   ~ 0
+3.3V_USB
+$Comp
+L C_Small C?
+U 1 1 5A429442
+P 3550 3300
+F 0 "C?" H 3560 3370 50  0000 L CNN
+F 1 "0.1uF" H 3560 3220 50  0000 L CNN
+F 2 "" H 3550 3300 50  0001 C CNN
+F 3 "" H 3550 3300 50  0001 C CNN
+	1    3550 3300
+	1    0    0    -1
+$EndComp
+$Comp
+L C_Small C?
+U 1 1 5A42947B
+P 3200 3300
+F 0 "C?" H 3210 3370 50  0000 L CNN
+F 1 "4.7uF" H 3210 3220 50  0000 L CNN
+F 2 "" H 3200 3300 50  0001 C CNN
+F 3 "" H 3200 3300 50  0001 C CNN
+	1    3200 3300
+	1    0    0    -1
+$EndComp
+$Comp
+L GND #PWR?
+U 1 1 5A4295A9
+P 3200 3550
+F 0 "#PWR?" H 3200 3300 50  0001 C CNN
+F 1 "GND" H 3200 3400 50  0000 C CNN
+F 2 "" H 3200 3550 50  0001 C CNN
+F 3 "" H 3200 3550 50  0001 C CNN
+	1    3200 3550
+	1    0    0    -1
+$EndComp
+$Comp
+L SP0503BAHTG U?
+U 1 1 5A42AB8B
+P 4650 4200
+F 0 "U?" H 4900 4450 60  0000 C CNN
+F 1 "SP0503BAHTG" H 4850 4050 60  0000 C CNN
+F 2 "TO_SOT_Packages_SMD:SOT-143" H 4650 3800 60  0001 C CNN
+F 3 "" H 4670 4220 60  0001 C CNN
+	1    4650 4200
+	1    0    0    -1
+$EndComp
+Wire Wire Line
+	4550 2450 4550 2500
+Wire Wire Line
+	4550 2500 4900 2500
+Wire Wire Line
+	5400 1650 5400 2200
+Wire Wire Line
+	5400 1650 6100 1650
+Wire Wire Line
+	5650 1650 5650 1700
+Wire Wire Line
+	6100 1650 6100 1700
+Connection ~ 5650 1650
+Wire Wire Line
+	5650 1900 5650 2000
+Wire Wire Line
+	5650 2000 6100 2000
+Wire Wire Line
+	6100 1900 6100 2050
+Wire Wire Line
+	4550 2250 4550 2150
+Wire Wire Line
+	4550 2150 5500 2150
+Connection ~ 5400 2150
+Wire Wire Line
+	5500 2150 5500 2200
+Connection ~ 6100 2000
+Wire Wire Line
+	3200 3200 3200 3100
+Wire Wire Line
+	3100 3100 4900 3100
+Wire Wire Line
+	3550 3200 3550 3100
+Connection ~ 3550 3100
+Wire Wire Line
+	3200 3400 3200 3550
+Wire Wire Line
+	3200 3500 3550 3500
+Wire Wire Line
+	3550 3500 3550 3400
+Connection ~ 3200 3500
+Connection ~ 3200 3100
+Wire Wire Line
+	4350 3500 4900 3500
+Wire Wire Line
+	4900 3600 4350 3600
+Wire Wire Line
+	4900 3400 4800 3400
+Wire Wire Line
+	4800 3100 4800 3800
+Connection ~ 4800 3100
+Wire Wire Line
+	4500 3500 4500 3800
+Connection ~ 4500 3500
+Wire Wire Line
+	4650 3800 4650 3600
+Connection ~ 4650 3600
+Connection ~ 4800 3400
+$Comp
+L GND #PWR?
+U 1 1 5A42AE08
+P 4500 4600
+F 0 "#PWR?" H 4500 4350 50  0001 C CNN
+F 1 "GND" H 4500 4450 50  0000 C CNN
+F 2 "" H 4500 4600 50  0001 C CNN
+F 3 "" H 4500 4600 50  0001 C CNN
+	1    4500 4600
+	1    0    0    -1
+$EndComp
+Wire Wire Line
+	4500 4500 4500 4600
+Wire Wire Line
+	4500 4550 5600 4550
+Wire Wire Line
+	5500 4550 5500 4000
+Connection ~ 4500 4550
+Wire Wire Line
+	5600 4550 5600 4000
+Connection ~ 5500 4550
+Wire Wire Line
+	6100 2800 6300 2800
+Wire Wire Line
+	6300 2900 6100 2900
+Wire Wire Line
+	6100 3500 6300 3500
+Wire Wire Line
+	6300 3600 6100 3600
+Wire Wire Line
+	6100 3700 6300 3700
 $EndSCHEMATC
