File: wireless_sensor.sch (KiCad schematic (older format))
At the start: 2 parts

Commit message: Files from laptop
Connections:
- net stm32l051k8t/PC14 renamed stm32l051k8t/PA4
- net stm32l051k8t/PC15 renamed stm32l051k8t/PA5
Changed lines of the file:
@@
 F3 "D-" B R 2200 1750 60
 F4 "VUSB" O R 2200 1850 60
-F5 "VSYS" O R 2200 1950 60
 $EndSheet
 $Sheet
-S 2800 1500 1050 600
+S 2800 1400 1050 700
 U 5A3B4F3A
 F0 "usb_serial" 60
@@
 F6 "STM_BL" O R 3850 1850 60
 F7 "VUSB" I L 2800 1850 60
+F8 "ESP_BL" O R 3850 1550 60
+F9 "STM_~RST~" O R 3850 1950 60
 $EndSheet
 $Comp
@@
 F3 "RX" I L 6850 1650 60
 F4 "WAKE" I L 6850 1850 60
-F5 "BOOTLOADER" I L 6850 1950 60
+F5 "BOOTLOADER" I R 7800 1650 60
 $EndSheet
 $Sheet
@@
 F16 "SW_1" I R 5850 4050 60
 F17 "ESP_WAKE" O R 5850 1850 60
-F18 "PC14" B R 5850 3350 60
-F19 "PC15" B R 5850 3450 60
+F18 "PA4" B R 5850 3350 60
+F19 "PA5" B R 5850 3450 60
 F20 "SDA" B R 5850 2850 60
 F21 "SCL" B R 5850 2950 60
-F22 "ESP_BL" O R 5850 1950 60
+F22 "~RST" I L 4500 1950 60
 $EndSheet
 $Sheet
@@
 $EndSheet
 $Sheet
-S 3250 3550 600  450
+S 3250 3450 600  500
 U 5A3BE733
 F0 "analog_filters" 60
@@
 F3 "AIN_2" O R 3850 3750 60
 F4 "AIN_3" O R 3850 3850 60
+F5 "AIN_0" O R 3850 3550 60
 $EndSheet
 Wire Wire Line
@@
 Wire Wire Line
 	2200 1850 2800 1850
-Wire Wire Line
-	2200 1950 2550 1950
-Wire Wire Line
-	2550 1950 2550 3350
 Wire Wire Line
 	6000 3350 5850 3350
@@
 	4500 3850 3850 3850
 Wire Wire Line
-	4500 3550 4300 3550
-Wire Wire Line
-	4300 3550 4300 3350
-Wire Wire Line
-	4300 3350 2550 3350
-Wire Wire Line
 	5850 2850 6850 2850
 Wire Wire Line
@@
 Wire Wire Line
 	6850 1850 5850 1850
-Wire Wire Line
-	5850 1950 6850 1950
 $Sheet
 S 6850 3750 950  650
@@
 Wire Wire Line
 	6850 4050 5850 4050
+Wire Wire Line
+	3850 3550 4500 3550
+Wire Wire Line
+	3850 1950 4500 1950
+Wire Wire Line
+	3850 1550 4150 1550
+Wire Wire Line
+	4150 1550 4150 1250
+Wire Wire Line
+	4150 1250 8000 1250
+Wire Wire Line
+	8000 1250 8000 1650
+Wire Wire Line
+	8000 1650 7800 1650
 $EndSCHEMATC
